File: node/lumin_node.kicad_pcb (KiCad board)
At the start: 2 copper layers, 50 x 50.1 mm, 17 parts, among them IC1 ATTINY441-SSU, P1 BUS_IN, P2 BUS_OUT, P3 LED_STRIP, Q1 Q_NMOS_GDS, Q2 Q_NMOS_GDS, Q3 Q_NMOS_GDS, U1 L7805CD2T-TR, U2 SN65HVD3082ED

Commit message: Shuffled PCB
Parts:
- Q1: value Q_NMOS_GDS -> LED_R
- Q2: value Q_NMOS_GDS -> LED_B
- Q3: value Q_NMOS_GDS -> LED_G
Routing:
- net GND: track 17.4 -> 23.1 mm, vias 6 -> 11
- net /LED_B_OUT: track 6.41 -> 9.29 mm
- net /LED_G_OUT: track 6.10 -> 8.92 mm
- net /LED_R_OUT: track 6.49 -> 8.49 mm
Other:
- outline, holes or cut-outs redrawn
